Commit message: walker_demo works now.

File: bioloid_description/urdf/typea.urdf (robot description, URDF)
Before this commit: robot typea, 25 links, 24 joints
Links:
- link l_ankle_lateral_link: geometry collision box size=0.0405 0.029 0.083; visual mesh filename=file:///home/robertkwan/catkin_ws/src/bioloid_common/bioloi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 scale=0.001 0.001 0.001
- link l_ankle_swing_link: geometry collision box size=0.051 0.0721 0.04; visual mesh filename=file:///home/robertkwan/catkin_ws/src/bioloid_common/bioloi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 scale=0.001 0.001 0.001
- link l_foot_link: geometry collision box size=0.009 0.061 0.101; visual mesh filename=file:///home/robertkwan/catkin_ws/src/bioloid_common/bioloi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 scale=0.001 0.001 0.001
- link l_hand_link: geometry collision box size=0.0131 0.0265 0.044; collision box size=0.0575 0.0175 0.035
- link l_hip_lateral_link: geometry collision box size=0.04 0.051 0.0721; visual mesh filename=file:///home/robertkwan/catkin_ws/src/bioloid_common/bioloi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 scale=0.001 0.001 0.001
- link l_hip_twist_link: geometry collision box size=0.029 0.083 0.0405; visual mesh filename=file:///home/robertkwan/catkin_ws/src/bioloid_common/bioloi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 scale=0.001 0.001 0.001
- link l_lower_arm_link: geometry collision box size=0.058 0.033 0.044; visual mesh filename=file:///home/robertkwan/catkin_ws/src/bioloid_common/bioloi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 scale=0.001 0.001 0.001
- link l_lower_leg_link: geometry collision box size=0.033 0.051 0.044; collision box size=0.067 0.03 0.049
- link l_shoulder_swing_link: geometry collision box size=0.052 0.039 0.036; visual mesh filename=file:///home/robertkwan/catkin_ws/src/bioloid_common/bioloi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 scale=0.001 0.001 0.001
- link l_upper_arm_link: geometry collision box size=0.047 0.033 0.052; collision box size=0.054 0.033 0.044
- link l_upper_leg_link: geometry collision box size=0.04 0.0371 0.049; collision box size=0.065 0.03 0.049
- link r_ankle_lateral_link: geometry collision box size=0.0405 0.029 0.083; visual mesh filename=file:///home/robertkwan/catkin_ws/src/bioloid_common/bioloi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 scale=0.001 0.001 0.001
- link r_ankle_swing_link: geometry collision box size=0.051 0.0721 0.04; visual mesh filename=file:///home/robertkwan/catkin_ws/src/bioloid_common/bioloi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 scale=0.001 0.001 0.001
- link r_foot_link: geometry collision box size=0.009 0.061 0.101; visual mesh filename=file:///home/robertkwan/catkin_ws/src/bioloid_common/bioloi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 scale=0.001 0.001 0.001
- link r_hand_link: geometry collision box size=0.0131 0.0265 0.044; collision box size=0.0575 0.0175 0.035
- link r_hip_lateral_link: geometry collision box size=0.04 0.051 0.0721; visual mesh filename=file:///home/robertkwan/catkin_ws/src/bioloid_common/bioloi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 scale=0.001 0.001 0.001
- link r_hip_twist_link: geometry collision box size=0.029 0.083 0.0405; visual mesh filename=file:///home/robertkwan/catkin_ws/src/bioloid_common/bioloi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 scale=0.001 0.001 0.001
- link r_lower_arm_link: geometry collision box size=0.058 0.033 0.044; visual mesh filename=file:///home/robertkwan/catkin_ws/src/bioloid_common/bioloi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 scale=0.001 0.001 0.001
- link r_lower_leg_link: geometry collision box size=0.033 0.051 0.044; collision box size=0.067 0.03 0.049
- link r_shoulder_swing_link: geometry collision box size=0.052 0.039 0.036; visual mesh filename=file:///home/robertkwan/catkin_ws/src/bioloid_common/bioloi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 scale=0.001 0.001 0.001
- link r_upper_arm_link: geometry collision box size=0.047 0.033 0.052; collision box size=0.054 0.033 0.044
- link r_upper_leg_link: geometry collision box size=0.04 0.0371 0.049; collision box size=0.065 0.03 0.049
- link torso_link: geometry collision box size=0.054 0.033 0.044; collision box size=0.065 0.099 0.043
